File: Receiver_Out_SMD/Outputs.kicad_sch (KiCad schematic)
At the start: 14 parts, among them J1 String1, J2 String2, J3 String3, J4 String4, U4 74HCT541

Commit message: new header
Parts:
- J1, J2, J3, J4: footprint Scotts:DG250-3.5-03P -> Scotts:PHOENIX_1864299; Digi-Key_PN 277-5737-ND/ED10555-ND -> 277-12185-ND; LCSC_PN C192778 -> C6394553; MPN 1843619/OSTTJ0311530 -> 1864299
Changed lines of the file:
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@@
 			)
 		)
-		(property "Footprint" "Scotts:DG250-3.5-03P"
+		(property "Footprint" "Scotts:PHOENIX_1864299"
 			(at 151.13 101.6 0)
 			(effects
@@
 			)
 		)
-		(property "Digi-Key_PN" "277-5737-ND/ED10555-ND"
+		(property "Digi-Key_PN" "277-12185-ND"
 			(at -36.322 -3.048 0)
 			(effects
@@
 			)
 		)
-		(property "MPN" "1843619/OSTTJ0311530"
+		(property "MPN" "1864299"
 			(at -36.322 -3.048 0)
 			(effects
@@
 			)
 		)
-		(property "LCSC_PN" "C192778"
+		(property "LCSC_PN" "C6394553"
 			(at 151.13 101.6 0)
 			(effects
@@
 			)
 		)
-		(property "Footprint" "Scotts:DG250-3.5-03P"
+		(property "Footprint" "Scotts:PHOENIX_1864299"
 			(at 162.56 101.6 0)
 			(effects
@@
 			)
 		)
-		(property "Digi-Key_PN" "277-5737-ND/ED10555-ND"
+		(property "Digi-Key_PN" "277-12185-ND"
 			(at -39.116 -2.794 0)
 			(effects
@@
 			)
 		)
-		(property "MPN" "1843619/OSTTJ0311530"
+		(property "MPN" "1864299"
 			(at -39.116 -2.794 0)
 			(effects
@@
 			)
 		)
-		(property "LCSC_PN" "C192778"
+		(property "LCSC_PN" "C6394553"
 			(at 162.56 101.6 0)
 			(effects
@@
 			)
 		)
-		(property "Footprint" "Scotts:DG250-3.5-03P"
+		(property "Footprint" "Scotts:PHOENIX_1864299"
 			(at 173.99 101.6 0)
 			(effects
@@
 			)
 		)
-		(property "Digi-Key_PN" "277-5737-ND/ED10555-ND"
+		(property "Digi-Key_PN" "277-12185-ND"
 			(at -38.354 -2.286 0)
 			(effects
@@
 			)
 		)
-		(property "MPN" "1843619/OSTTJ0311530"
+		(property "MPN" "1864299"
 			(at -38.354 -2.286 0)
 			(effects
@@
 			)
 		)
-		(property "LCSC_PN" "C192778"
+		(property "LCSC_PN" "C6394553"
 			(at 173.99 101.6 0)
 			(effects
@@
 			)
 		)
-		(property "Footprint" "Scotts:DG250-3.5-03P"
+		(property "Footprint" "Scotts:PHOENIX_1864299"
 			(at 185.42 101.6 0)
 			(effects
@@
 			)
 		)
-		(property "Digi-Key_PN" "277-5737-ND/ED10555-ND"
+		(property "Digi-Key_PN" "277-12185-ND"
 			(at -36.068 -2.032 0)
 			(effects
@@
 			)
 		)
-		(property "MPN" "1843619/OSTTJ0311530"
+		(property "MPN" "1864299"
 			(at -36.068 -2.032 0)
 			(effects
@@
 			)
 		)
-		(property "LCSC_PN" "C192778"
+		(property "LCSC_PN" "C6394553"
 			(at 185.42 101.6 0)
 			(effects
