File: SM_Receiver_Out_SMD/Diff_In.kicad_sch (KiCad schematic)
At the start: 14 parts

Commit message: 2026 updates
Parts:
- added JP1: Serial_PWR, Jumper:SolderJumper-3_P2.0mm_Open_TrianglePad1.0x1.5mm, symbol Jumper:SolderJumper_3_Open
- C4: value (none) -> 0.1uF; footprint (none) -> Capacitor_SMD:C_0603_1608Metric_Pad1.08x0.95mm_HandSolder
- J7, J8: value (none) -> RJ45; footprint (none) -> Connector_RJ:RJ45_Amphenol_54602-x08_Horizontal
- R12, R13, R14, R15: value (none) -> 100ohm; footprint (none) -> Resistor_SMD:R_0603_1608Metric_Pad0.98x0.95mm_HandSolder
- R2: value (none) -> 100K; footprint (none) -> Resistor_SMD:R_0603_1608Metric_Pad0.98x0.95mm_HandSolder
- R3, R4, R5, R6: value (none) -> 120; footprint (none) -> Resistor_SMD:R_0603_1608Metric_Pad0.98x0.95mm_HandSolder
- SW2: value (none) -> Terminators; footprint (none) -> Button_Switch_THT:SW_DIP_SPSTx04_Slide_6.7x11.72mm_W7.62mm_P2.54mm_LowProfile
- U3: value (none) -> AM26LV32; footprint (none) -> Package_SO:SOIC-16_3.9x9.9mm_P1.27mm; Digi-Key_PN 296-37322-1-ND -> 296-18090-1-ND; LCSC_PN C6180 -> C527448; MPN AM26C32INSR -> AM26LV32IDR
Connections:
- net +3V3: now also JP1.3 (B); no longer C4.1, U3.16 (VCC)
- new net: C4.1, JP1.2 (C), U3.16 (VCC)
- new net +5V: JP1.1 (A)
Other:
- moved on the sheet: C4
