File: SM_Receiver_Out_SMD/Micro.kicad_sch (KiCad schematic)
At the start: 22 parts

Commit message: 2026 updates
Parts:
- added TP9: DIFF_EN, TestPoint:TestPoint_Pad_D1.5mm, symbol Connector:TestPoint
- C5: value (none) -> 0.1uF; footprint (none) -> Capacitor_SMD:C_0603_1608Metric_Pad1.08x0.95mm_HandSolder
- D4: value (none) -> LED; footprint (none) -> LED_SMD:LED_0603_1608Metric_Pad1.05x0.95mm_HandSolder
- J10: value (none) -> SWD; footprint (none) -> Scotts:1x02_Horizontal_SMD
- J5: value (none) -> OLED; footprint (none) -> OLED-SSD1306-128X64-I2C:OLED-SSD1306-128X64-I2C-THT
- J9: value (none) -> Debug; footprint (none) -> Connector_PinHeader_2.54mm:PinHeader_1x03_P2.54mm_Vertical
- R11: value (none) -> 220; footprint (none) -> Resistor_SMD:R_0603_1608Metric_Pad0.98x0.95mm_HandSolder
- R16, R17, R18, R19: value (none) -> 100ohm; footprint (none) -> Resistor_SMD:R_0603_1608Metric_Pad0.98x0.95mm_HandSolder
- SW1: value (none) -> ID; footprint (none) -> Button_Switch_THT:Nidec_Copal_SH-7010C
- SW3: value (none) -> User; footprint (none) -> Scotts:SW_Push_1P1T_NO_6x6mm_H9.5mm
- SW4: value (none) -> RUN; footprint (none) -> Scotts:SW_Push_1P1T_NO_6x6mm_H9.5mm
- TP1: value (none) -> DATA1; footprint (none) -> TestPoint:TestPoint_Pad_D1.5mm
- TP2: value (none) -> DATA2; footprint (none) -> TestPoint:TestPoint_Pad_D1.5mm
- TP3: value (none) -> DATA3; footprint (none) -> TestPoint:TestPoint_Pad_D1.5mm
- TP4: value (none) -> DATA4; footprint (none) -> TestPoint:TestPoint_Pad_D1.5mm
- TP5: value (none) -> EN1; footprint (none) -> TestPoint:TestPoint_Pad_D1.5mm
- TP6: value (none) -> EN2; footprint (none) -> TestPoint:TestPoint_Pad_D1.5mm
- TP7: value (none) -> EN3; footprint (none) -> TestPoint:TestPoint_Pad_D1.5mm
- TP8: value (none) -> EN4; footprint (none) -> TestPoint:TestPoint_Pad_D1.5mm
- U1: value (none) -> Pico; footprint (none) -> MCU_RaspberryPi_and_Boards:RPi_Pico_SMD_TH
Connections:
- net DIFF_EN: now also TP9.1
Other:
- moved on the sheet: TP5, TP6, TP7, TP8
