File: SM_Receiver_Out_SMD/Outputs.kicad_sch (KiCad schematic)
At the start: 17 parts

Commit message: 2026 updates
Parts:
- C3: value (none) -> 0.1uF; footprint (none) -> Capacitor_SMD:C_0603_1608Metric_Pad1.08x0.95mm_HandSolder
- F1, F2, F3, F4: value (none) -> 3544-2; footprint (none) -> Scotts:FUSE_3544-2
- J1: value (none) -> String1; footprint (none) -> Connector_Phoenix_MC:PhoenixContact_MCV_1,5_3-G-3.5_1x03_P3.50mm_Vertical
- J2: value (none) -> String2; footprint (none) -> Connector_Phoenix_MC:PhoenixContact_MCV_1,5_3-G-3.5_1x03_P3.50mm_Vertical
- J3: value (none) -> String3; footprint (none) -> Connector_Phoenix_MC:PhoenixContact_MCV_1,5_3-G-3.5_1x03_P3.50mm_Vertical
- J4: value (none) -> String4; footprint (none) -> Connector_Phoenix_MC:PhoenixContact_MCV_1,5_3-G-3.5_1x03_P3.50mm_Vertical
- R10, R7, R8, R9: value (none) -> 33ohm; footprint (none) -> Resistor_SMD:R_0603_1608Metric_Pad0.98x0.95mm_HandSolder
- U4, U5, U6, U7: value (none) -> 74AHCT1G125; footprint (none) -> Package_SO:TSOP-5_1.65x3.05mm_P0.95mm
