File: SM_Receiver_Out_SMD/Receiver_Out.kicad_pcb (KiCad board)
At the start: 2 copper layers, 83.2 x 71.4 mm, 67 parts, among them J1 String1, J10 SWD, J2 String2, J3 String3, J4 String4, J5 OLED, J6 VIN_Voltage, J7 RJ45, J8 RJ45, J9 Debug, SW1 ID, SW2 Terminators, SW3 User, SW4 RUN, U1 Pico, U2 AMS1117-5.0, U3 AM26C32IN, U4 74AHCT1G125, U5 74AHCT1G125, U6 74AHCT1G125, U7 74AHCT1G125

Commit message: 2026 updates
Parts:
- removed REF**: KiCad-Logo2_6mm_SilkScreen, Symbol:KiCad-Logo2_6mm_SilkScreen
- added JP1: Serial_PWR, Jumper:SolderJumper-3_P2.0mm_Open_TrianglePad1.0x1.5mm, B.Cu at (58.0, 149.3)
- added TP9: DIFF_EN, TestPoint:TestPoint_Pad_D1.5mm, B.Cu at (73.2, 139.4)
- H1, H2, H3, H4: footprint Scotts:MountingHole_3.7mm -> MountingHole:MountingHole_3.7mm
- U3: value AM26C32IN -> AM26LV32
- moved G*** 33.1 mm to (58.6, 114.0)
- moved R11 7.71 mm to (60.7, 145.0), turned to 180 degrees
- moved J9 2.50 mm to (70.0, 147.5)
- moved C5 1.68 mm to (45.8, 138.8), turned to 90 degrees
- moved D4 0.98 mm to (64.4, 145.0), turned to 0 degrees
Connections:
- C4 pad 1: +3V3 -> Net-(JP1-C)
- U3 pad 16: +3V3 -> Net-(JP1-C)
Routing:
- net Net-(JP1-C): track 0.00 -> 51.7 mm, vias 0 -> 3
- net +3V3: track 105.6 -> 89.2 mm, vias 2 -> 1
- net +5V: track 150.0 -> 162.8 mm
- net Net-(J9-Pin_2): track 12.5 -> 5.44 mm
- net GND: track 0.00 -> 4.37 mm, vias 105 -> 96
- net Net-(J9-Pin_1): track 14.6 -> 11.7 mm
- net Net-(U1-RUN): track 107.3 -> 109.4 mm
- net Serial4_P: track 61.5 -> 59.7 mm
- net Net-(D4-A): track 26.3 -> 24.7 mm
- net Serial3_P: track 52.8 -> 51.6 mm
- net /Micro/SDA: track 50.6 -> 49.6 mm
- net /Micro/SCL: track 53.9 -> 54.7 mm
Other:
- board text added: "3V"
- board text added: "5V"
