File: SM_Receiver_Out_SMD/Receiver_Out.kicad_sch (KiCad schematic)
At the start: 12 parts

Commit message: 2026 updates
Parts:
- C1, C2: value (none) -> 10uF; footprint (none) -> Capacitor_SMD:C_0805_2012Metric_Pad1.18x1.45mm_HandSolder
- D1: value (none) -> B5819W; footprint (none) -> Diode_SMD:D_SOD-123
- D2: value (none) -> VIN LED; footprint (none) -> LED_SMD:LED_0603_1608Metric_Pad1.05x0.95mm_HandSolder
- H1, H2, H3, H4: value (none) -> MountingHole; footprint (none) -> MountingHole:MountingHole_3.7mm
- J6: value (none) -> VIN_Voltage; footprint (none) -> Connector_PinHeader_2.54mm:PinHeader_1x03_P2.54mm_Vertical
- R1: value (none) -> 1K; footprint (none) -> Resistor_SMD:R_0603_1608Metric_Pad0.98x0.95mm_HandSolder
- TB1: value (none) -> Power In; footprint (none) -> Barrier_Blocks:BARRIER_BLOCK_1ROW_2POS
- U2: value (none) -> AMS1117-5.0; footprint (none) -> Package_TO_SOT_SMD:SOT-223-3_TabPin2
